File: PCBfirst.sch (KiCad schematic (older format))
At the start: 24 parts, among them SW1 SW_Push, U1 ATmega32U4-AU, Y1 16MHz

Commit message: fixed! on to making pcb
i set the footprint library of the kicad wrong.
Parts:
- MX1, MX2, MX3, MX4: footprint (none) -> MX_Alps_Hybrid:MX-1U
Changed lines of the file:
@@
 EESchema Schematic File Version 4
+LIBS:PCBfirst-cache
 EELAYER 30 0
 EELAYER END
@@
 F 0 "MX1" H 7033 2773 60  0000 C CNN
 F 1 "MX-NoLED" H 7033 2699 20  0000 C CNN
-F 2 "" H 6375 2525 60  0001 C CNN
+F 2 "MX_Alps_Hybrid:MX-1U" H 6375 2525 60  0001 C CNN
 F 3 "" H 6375 2525 60  0001 C CNN
 	1    7000 2550
@@
 F 0 "MX2" H 7633 2773 60  0000 C CNN
 F 1 "MX-NoLED" H 7633 2699 20  0000 C CNN
-F 2 "" H 6975 2525 60  0001 C CNN
+F 2 "MX_Alps_Hybrid:MX-1U" H 6975 2525 60  0001 C CNN
 F 3 "" H 6975 2525 60  0001 C CNN
 	1    7600 2550
@@
 F 0 "MX3" H 7183 3573 60  0000 C CNN
 F 1 "MX-NoLED" H 7183 3499 20  0000 C CNN
-F 2 "" H 6525 3325 60  0001 C CNN
+F 2 "MX_Alps_Hybrid:MX-1U" H 6525 3325 60  0001 C CNN
 F 3 "" H 6525 3325 60  0001 C CNN
 	1    7150 3350
@@
 F 0 "MX4" H 7733 3573 60  0000 C CNN
 F 1 "MX-NoLED" H 7733 3499 20  0000 C CNN
-F 2 "" H 7075 3325 60  0001 C CNN
+F 2 "MX_Alps_Hybrid:MX-1U" H 7075 3325 60  0001 C CNN
 F 3 "" H 7075 3325 60  0001 C CNN
 	1    7700 3350
